Commit message: Updated CAD Model

File: src/rogue/description/urdf/rogue_des.urdf (robot description, URDF)
Before this commit: robot rogue, 8 links, 7 joints
Links:
- removed link chassis_link
- link Driving_Front_Left_Link: mass 1.39036444547767 -> 3.92591214810011; geometry collision mesh filename=package://rogue/meshes/Driving_Front_Left_Link.STL; visual mesh filename=package://rogue/meshes/Driving_Front_Left_Link.STL
- link Driving_Front_Right_Link: mass 1.39036444547767 -> 3.92591214810005; geometry collision mesh filename=package://rogue/meshes/Driving_Front_Right_Link.STL; visual mesh filename=package://rogue/meshes/Driving_Front_Right_Link.STL
- link Driving_Left_Link: mass 1.3904 -> 3.9259121481001; geometry collision mesh filename=package://rogue/meshes/Driving_Left_Link.STL; visual mesh filename=package://rogue/meshes/Driving_Left_Link.STL
- link Driving_Right_Link: mass 1.3904 -> 3.92591214810012; geometry collision mesh filename=package://rogue/meshes/Driving_Right_Link.STL; visual mesh filename=package://rogue/meshes/Driving_Right_Link.STL
- link Steering_Front_Left_Link: mass 0.291764052989946 -> 1.85682341940371; geometry collision mesh filename=package://rogue/meshes/Steering_Front_Left_Link.STL; visual mesh filename=package://rogue/meshes/Steering_Front_Left_Link.STL
- link Steering_Front_Right_Link: mass 0.291764052989947 -> 1.85682341940371; geometry collision mesh filename=package://rogue/meshes/Steering_Front_Right_Link.STL; visual mesh filename=package://rogue/meshes/Steering_Front_Right_Link.STL
- link base_link: mass None -> 7.01937426124387; geometry collision mesh filename=package://rogue/meshes/base_link.STL; visual mesh filename=package://rogue/meshes/base_link.STL
Joints:
- removed joint base_joint
- joint Driving_Front_Left: axis 0.99823 0 0.059504 -> 0 0.309764314615681 -0.95081337253463; limit lower=-100 upper=100 effort=0 velocity=4.05 -> (none); origin xyz=0 -0.1145 0 rpy=1.1343 -0.031639 0.054039 -> xyz=0 0.105281491318534 0 rpy=1.25585118201626 0 3.14159265358979
- joint Driving_Front_Right: axis 0.99823 0 0.059504 -> 0 0.294142720525736 0.955761507888719; limit lower=-100 upper=100 effort=0 velocity=4.05 -> (none); origin xyz=0 -0.1145 0 rpy=1.5327 -0.054583 0.059592 -> xyz=0 -0.10690236537747 0 rpy=-1.27223789169551 0 3.14159265358979
- joint Driving_Left: axis 0.99823 0 0.059504 -> 1 0 0; limit lower=-100 upper=100 effort=0 velocity=4.05 -> (none); origin xyz=-0.56821 0.2102 -0.1145 rpy=-2.0317 -0.026508 1.4579 -> xyz=0.535731179493507 -0.407500000000434 -0.49861768424532 rpy=1.96681303566779 0 1.5707963267949; parent chassis_link -> base_link
- joint Driving_Right: axis 0.99823 0 0.059504 -> 1 0 0; limit lower=-100 upper=100 effort=0 velocity=4.05 -> (none); origin xyz=-0.55679 -0.2102 -0.1145 rpy=-2.0317 -0.026508 -1.6837 -> xyz=0.536022919102397 0 -0.498234906342967 rpy=-1.8359994985479 0 -1.5707963267949; parent chassis_link -> base_link
- joint Steering_Front_Left: limit lower=-3.14 upper=3.14 effort=0 velocity=4.05 -> (none); origin xyz=0.5625 0.306 0 rpy=1.5708 0 1.568 -> xyz=-0.539929731609329 -0.542999999999972 -0.193804668520646 rpy=-1.5789896816345 0 -1.5707963267949; parent chassis_link -> base_link
- joint Steering_Front_Right: limit lower=-3.14 upper=3.14 effort=0 velocity=4.05 -> (none); origin xyz=0.5625 -0.306 0 rpy=1.5708 0 -1.5736 -> xyz=-0.539856087012609 0.0730000000000078 -0.194276018002367 rpy=1.57827537993681 0 1.5707963267949; parent chassis_link -> base_link

File: src/rogue/description/urdf/rogue_des.xacro (robot description, xacro)
@@ -4,6 +4,8 @@
 <!-- |    EDITING THIS FILE BY HAND IS NOT RECOMMENDED                                 | -->
 <!-- =================================================================================== -->
+<!-- This URDF was automatically created by SolidWorks to URDF Exporter! Originally created by Stephen Brawner (brawner@gmail.com)
+     Commit Version: 1.6.0-4-g7f85cfe  Build Version: 1.6.7995.38578
+     For more information, please see http://wiki.ros.org/sw_urdf_exporter -->
 <robot name="rogue">
-  <!-- base link -->
   <link name="base_link">
     <origin rpy="0 0 0" xyz="0 0 0"/>
@@ -13,5 +15,5 @@
     <parent link="base_link"/>
     <child link="chassis_link"/>
-    <origin xyz="0 0 0"/>
+    <origin xyz="0 -0.235 -0.11"/>
   </joint>
   <!-- chassis link -->
@@ -20,16 +22,17 @@
       <origin rpy="0 0 0" xyz="-0.00246940894159626 0.1058972543147 5.46494556407368E-17"/>
       <mass value="136.620754096564"/>
-      <inertia ixx="3.3220316255083" ixy="1.43783842796417E-19" ixz="8.74036870867536E-05" iyy="20.3007194974988" iyz="3.4410713482206E-19" izz="18.0177890671193"/>
-    </inertial>
-    <visual>
+      <inertia ixx="0.07413" ixy="-0.00011285" ixz="-1.4435E-06" iyy="0.14749" iyz="1.7539E-08" izz="0.11937"/>
+    </inertial>
+    <visual>
+    <origin rpy="0 0 0" xyz="0 0.235 0.11"/>
       <geometry>
         <mesh filename="package://rogue/description/meshes/base_link.stl"/>
       </geometry>
       <material name="">
-        <color rgba="0.792156862745098 0.819607843137255 0.933333333333333 1"/>
-      </material>
-    </visual>
-    <collision>
-      <origin rpy="0 0 0" xyz="0 0 0"/>
+        <color rgba="0.79216 0.81961 0.93333 1"/>
+      </material>
+    </visual>
+    <collision>
+      <origin rpy="0 0 0" xyz="0 0.235 0.11"/>
       <geometry>
         <mesh filename="package://rogue/description/meshes/base_link.stl"/>
@@ -37,177 +40,171 @@
     </collision>
   </link>
-  <!-- joint chassis ST front_left -->
+  <link name="Steering_Front_Left_Link">
+    <inertial>
+      <origin rpy="0 0 0" xyz="-0.00974656428371329 0.171466468601951 3.33066907387547E-15"/>
+      <mass value="1.85682341940371"/>
+      <inertia ixx="0.0307102115747056" ixy="0.00225357611286934" ixz="1.56419202677199E-14" iyy="0.0217734903548105" iyz="-1.09535590233495E-15" izz="0.0500272192704002"/>
+    </inertial>
+    <visual>
+      <origin rpy="0 0 0" xyz="0 0 0"/>
+      <geometry>
+        <mesh filename="package://rogue/description/meshes/Steering_Front_Left_Link.stl"/>
+      </geometry>
+      <material name="">
+        <color rgba="0.666666666666667 0.698039215686274 0.768627450980392 1"/>
+      </material>
+    </visual>
+    <collision>
+      <origin rpy="0 0 0" xyz="0 0 0"/>
+      <geometry>
+        <mesh filename="package://rogue/description/meshes/Steering_Front_Left_Link.stl"/>
+      </geometry>
+    </collision>
+  </link>
   <joint name="Steering_Front_Left" type="continuous">
-    <parent link="chassis_link"/>
+    <origin rpy="-1.5789896816345 0 -1.5707963267949" xyz="-0.539929731609329 -0.307999999999972 -0.0838046685206459"/>
+    <parent link="base_link"/>
     <child link="Steering_Front_Left_Link"/>
-    <origin rpy="1.5708 0 1.568" xyz="0.5625 0.306 0"/>
     <axis xyz="0 1 0"/>
-    <limit effort="0" lower="-3.14" upper="3.14" velocity="4.05"/>
-  </joint>
-  <!-- link ST front left -->
-  <link name="Steering_Front_Left_Link">
-    <inertial>
-      <origin rpy="0 0 0" xyz="0.0265509625988199 -0.0902801904129602 0.00150839438422112"/>
-      <mass value="0.291764052989946"/>
-      <inertia ixx="0.000897400695611327" ixy="-0.000181864873221569" ixz="-4.0471931325247E-05" iyy="0.000964137142000603" iyz="-1.0331977698871E-05" izz="0.00160749385918111"/>
-    </inertial>
-    <visual>
-      <origin rpy="0 0 0" xyz="0 0 0"/>
-      <geometry>
-        <mesh filename="package://rogue/description/meshes/Steering_Front_Left_Link.stl"/>
-      </geometry>
-      <material name="">
-        <color rgba="0.44313725490196076 0.6235294117647059 0.5686274509803921 1.0"/>
-      </material>
-    </visual>
-    <collision>
-      <origin rpy="0 0 0" xyz="0 0 0"/>
-      <geometry>
-        <mesh filename="package://rogue/description/meshes/Steering_Front_Left_Link.stl"/>
-      </geometry>
-    </collision>
-  </link>
-  <!-- joint ST front left DR front_left -->
+  </joint>
+  <link name="Driving_Front_Left_Link">
+    <inertial>
+      <origin rpy="0 0 0" xyz="0.000635564712824666 -0.152689840468291 -0.00010385666276358"/>
+      <mass value="3.92591214810011"/>
+      <inertia ixx="0.040527651338497" ixy="8.45389473885711E-07" ixz="-3.83041768788121E-09" iyy="0.0313134736150526" iyz="8.54177538313404E-06" izz="0.0312863477526415"/>
+    </inertial>
+    <visual>
+      <origin rpy="0 0 0" xyz="0 0.148 0"/>
+      <geometry>
+        <mesh filename="package://rogue/description/meshes/Driving_Front_Left_Link.stl"/>
+      </geometry>
+      <material name="">
+        <color rgba="0.792156862745098 0.819607843137255 0.933333333333333 1"/>
+      </material>
+    </visual>
+    <collision>
+      <origin rpy="0 0 0" xyz="0 0.148 0"/>
+      <geometry>
+        <mesh filename="package://rogue/description/meshes/Driving_Front_Left_Link.stl"/>
+      </geometry>
+    </collision>
+  </link>
   <joint name="Driving_Front_Left" type="continuous">
+    <origin rpy="0 0 3.14159265358979" xyz="0 ${0.14261211817947+0.148} 0"/>
     <parent link="Steering_Front_Left_Link"/>
     <child link="Driving_Front_Left_Link"/>
-    <origin rpy="1.1343 -0.031639 0.054039" xyz="0 -0.1145 0"/>
-    <axis xyz="0.99823 0 0.059504"/>
-    <limit effort="0" lower="-100" upper="100" velocity="4.05"/>
-  </joint>
-  <!-- link DR front_left -->
-  <link name="Driving_Front_Left_Link">
-    <inertial>
-      <origin rpy="0 0 0" xyz="-0.0182564505721252 -3.92727932868597E-06 -0.00112517178645061"/>
-      <mass value="1.39036444547767"/>
-      <inertia ixx="0.00504431627608896" ixy="6.66802588932824E-07" ixz="3.18555927896634E-05" iyy="0.00451167026228943" iyz="-2.22813617032334E-07" izz="0.00451213600378384"/>
-    </inertial>
-    <visual>
-      <origin rpy="0 0 0" xyz="0 0 0"/>
-      <geometry>
-        <mesh filename="package://rogue/description/meshes/Driving_Front_Left_Link.stl"/>
-      </geometry>
-    </visual>
-    <collision>
-      <origin rpy="0 0 0" xyz="0 0 0"/>
-      <geometry>
-        <mesh filename="package://rogue/description/meshes/Driving_Front_Left_Link.stl"/>
-      </geometry>
-    </collision>
-  </link>
-  <!-- joint chassis ST right -->
+    <axis xyz="1 0 0"/>
+  </joint>
+  <link name="Steering_Front_Right_Link">
+    <inertial>
+      <origin rpy="0 0 0" xyz="-0.00974656428371296 -0.171380762932291 -8.54871728961371E-15"/>
+      <mass value="1.85682341940371"/>
+      <inertia ixx="0.0307102115747056" ixy="-0.00225357611286932" ixz="-1.57031471972793E-14" iyy="0.0217734903548105" iyz="-1.99752053006014E-15" izz="0.0500272192704002"/>
+    </inertial>
+    <visual>
+      <origin rpy="0 0 0" xyz="0 0 0"/>
+      <geometry>
+        <mesh filename="package://rogue/description/meshes/Steering_Front_Right_Link.stl"/>
+      </geometry>
+      <material name="">
+        <color rgba="0.666666666666667 0.698039215686274 0.768627450980392 1"/>
+      </material>
+    </visual>
+    <collision>
+      <origin rpy="0 0 0" xyz="0 0 0"/>
+      <geometry>
+        <mesh filename="package://rogue/description/meshes/Steering_Front_Right_Link.stl"/>
+      </geometry>
+    </collision>
+  </link>
   <joint name="Steering_Front_Right" type="continuous">
-    <parent link="chassis_link"/>
+    <origin rpy="1.57827537993681 0 1.5707963267949" xyz="-0.539856087012609 0.308000000000008 -0.0842760180023664"/>
+    <parent link="base_link"/>
     <child link="Steering_Front_Right_Link"/>
-    <origin rpy="1.5708 0 -1.5736" xyz="0.5625 -0.306 0"/>
     <axis xyz="0 1 0"/>
-    <limit effort="0" lower="-3.14" upper="3.14" velocity="4.05"/>
-  </joint>
-  <!-- link ST front_right -->
-  <link name="Steering_Front_Right_Link">
-    <inertial>
-      <origin rpy="0 0 0" xyz="0.0265509625988167 -0.0902801904129674 0.00150839438421835"/>
-      <mass value="0.291764052989947"/>
-      <inertia ixx="0.000897400695611324" ixy="-0.00018186487322157" ixz="-4.04719313252156E-05" iyy="0.000964137142000604" iyz="-1.03319776988643E-05" izz="0.00160749385918111"/>
-    </inertial>
-    <visual>
-      <origin rpy="0 0 0" xyz="0 0 0"/>
-      <geometry>
-        <mesh filename="package://rogue/description/meshes/Steering_Front_Right_Link.stl"/>
-      </geometry>
-      <material name="">
-        <color rgba="0.44313725490196076 0.6235294117647059 0.5686274509803921 1.0"/>
-      </material>
-    </visual>
-    <collision>
-      <origin rpy="0 0 0" xyz="0 0 0"/>
-      <geometry>
-        <mesh filename="package://rogue/description/meshes/Steering_Front_Right_Link.stl"/>
-      </geometry>
-    </collision>
-  </link>
-  <!-- joint ST front right DR right -->
+  </joint>
+  <link name="Driving_Front_Right_Link">
+    <inertial>
+      <origin rpy="0 0 0" xyz="0.000635564712824388 0.152474662096144 0.000103856662758472"/>
+      <mass value="3.92591214810005"/>
+      <inertia ixx="0.0405276513384967" ixy="-8.45389473903581E-07" ixz="3.83041770842588E-09" iyy="0.0313134736150523" iyz="8.54177538309055E-06" izz="0.0312863477526412"/>
+    </inertial>
+    <visual>
+      <origin rpy="0 0 0" xyz="0 -0.148 0"/>
+      <geometry>
+        <mesh filename="package://rogue/description/meshes/Driving_Front_Right_Link.stl"/>
+      </geometry>
+      <material name="">
+        <color rgba="0.792156862745098 0.819607843137255 0.933333333333333 1"/>
+      </material>
+    </visual>
+    <collision>
+      <origin rpy="0 0 0" xyz="0 -0.148 0"/>
+      <geometry>
+        <mesh filename="package://rogue/description/meshes/Driving_Front_Right_Link.stl"/>
+      </geometry>
+    </collision>
+  </link>
   <joint name="Driving_Front_Right" type="continuous">
+    <origin rpy="0 0 3.14159265358979" xyz="0 ${-0.142741590881956-0.148} 0"/>
     <parent link="Steering_Front_Right_Link"/>
     <child link="Driving_Front_Right_Link"/>
-    <origin rpy="1.5327 -0.054583 0.059592" xyz="0 -0.1145 0"/>
-    <axis xyz="0.99823 0 0.059504"/>
-    <limit effort="0" lower="-100" upper="100" velocity="4.05"/>
-  </joint>
-  <!-- link DR front_right -->
-  <link name="Driving_Front_Right_Link">
-    <inertial>
-      <origin rpy="0 0 0" xyz="-0.0182564505721275 -3.92727933196113E-06 -0.00112517178645236"/>
-      <mass value="1.39036444547767"/>
-      <inertia ixx="0.00504431627608894" ixy="6.66802588895595E-07" ixz="3.18555927896797E-05" iyy="0.00451167026228944" iyz="-2.22813616974866E-07" izz="0.00451213600378381"/>
-    </inertial>
-    <visual>
-      <origin rpy="0 0 0" xyz="0 0 0"/>
-      <geometry>
-        <mesh filename="package://rogue/description/meshes/Driving_Front_Right_Link.stl"/>
-      </geometry>
-    </visual>
-    <collision>
-      <origin rpy="0 0 0" xyz="0 0 0"/>
-      <geometry>
-        <mesh filename="package://rogue/description/meshes/Driving_Front_Right_Link.stl"/>
-      </geometry>
-    </collision>
-  </link>
-  <!-- joint chassis DR_left -->
+    <axis xyz="1 0 0"/>
+  </joint>
+  <link name="Driving_Left_Link">
+    <inertial>
+      <origin rpy="0 0 0" xyz="-0.134864435287178 0.000687652998535182 -0.000103856662875601"/>
+      <mass value="3.9259121481001"/>
+      <inertia ixx="0.0405276513384971" ixy="8.45389473657967E-07" ixz="-3.83041783364525E-09" iyy="0.0313134736150526" iyz="8.54177538309626E-06" izz="0.0312863477526416"/>
+    </inertial>
+    <visual>
+      <origin rpy="0 0 0" xyz="0 0 0"/>
+      <geometry>
+        <mesh filename="package://rogue/description/meshes/Driving_Left_Link.stl"/>
+      </geometry>
+      <material name="">
+        <color rgba="0.792156862745098 0.819607843137255 0.933333333333333 1"/>
+      </material>
+    </visual>
+    <collision>
+      <origin rpy="0 0 0" xyz="0 0 0"/>
+      <geometry>
+        <mesh filename="package://rogue/description/meshes/Driving_Left_Link.stl"/>
+      </geometry>
+    </collision>
+  </link>
   <joint name="Driving_Left" type="continuous">
-    <parent link="chassis_link"/>
+    <origin rpy="1.5707963267949 0 1.5707963267949" xyz="0.535731179493507 -0.172500000000432 -0.38861768424532"/>
+    <parent link="base_link"/>
     <child link="Driving_Left_Link"/>
-    <origin rpy="-2.0317 -0.026508 1.4579" xyz="-0.56821 0.2102 -0.1145"/>
-    <axis xyz="0.99823 0 0.059504"/>
-    <limit effort="0" lower="-100" upper="100" velocity="4.05"/>
-  </joint>
-  <!-- link DR left -->
-  <link name="Driving_Left_Link">
-    <inertial>
-      <origin rpy="0 0 0" xyz="0.077549 -3.9273E-06 0.0045857"/>
-      <mass value="1.3904"/>
-      <inertia ixx="0.0050443" ixy="6.668E-07" ixz="3.1856E-05" iyy="0.0045117" iyz="-2.2281E-07" izz="0.0045121"/>
-    </inertial>
-    <visual>
-      <origin rpy="0 0 0" xyz="0 0 0"/>
-      <geometry>
-        <mesh filename="package://rogue/description/meshes/Driving_Left_Link.stl"/>
-      </geometry>
-    </visual>
-    <collision>
-      <origin rpy="0 0 0" xyz="0 0 0"/>
-      <geometry>
-        <mesh filename="package://rogue/description/meshes/Driving_Left_Link.stl"/>
-      </geometry>
-    </collision>
-  </link>
-  <!-- joint chassis DR_right -->
+    <axis xyz="1 0 0"/>
+  </joint>
+  <link name="Driving_Right_Link">
+    <inertial>
+      <origin rpy="0 0 0" xyz="-0.134864435287174 -0.000687652998533683 0.00010385666287549"/>
+      <mass value="3.92591214810012"/>
+      <inertia ixx="0.0405276513384973" ixy="-8.45389473982144E-07" ixz="3.83041772531102E-09" iyy="0.0313134736150526" iyz="8.54177538295617E-06" izz="0.0312863477526417"/>
+    </inertial>
+    <visual>
+      <origin rpy="0 0 0" xyz="0 0 0"/>
+      <geometry>
+        <mesh filename="package://rogue/description/meshes/Driving_Right_Link.stl"/>
+      </geometry>
+      <material name="">
+        <color rgba="0.792156862745098 0.819607843137255 0.933333333333333 1"/>
+      </material>
+    </visual>
+    <collision>
+      <origin rpy="0 0 0" xyz="0 0 0"/>
+      <geometry>
+        <mesh filename="package://rogue/description/meshes/Driving_Right_Link.stl"/>
+      </geometry>
+    </collision>
+  </link>
   <joint name="Driving_Right" type="continuous">
-    <parent link="chassis_link"/>
+    <origin rpy="-1.5707963267949 0 -1.5707963267949" xyz="0.536022919102346 0.17249999999957 -0.388234906342967"/>
+    <parent link="base_link"/>
     <child link="Driving_Right_Link"/>
-    <origin rpy="-2.0317 -0.026508 -1.6837" xyz="-0.55679 -0.2102 -0.1145"/>
-    <axis xyz="0.99823 0 0.059504"/>
-    <limit effort="0" lower="-100" upper="100" velocity="4.05"/>
-  </joint>
-  <!-- link DR right -->
-  <link name="Driving_Right_Link">
-    <inertial>
-      <origin rpy="0 0 0" xyz="0.077549 -3.9273E-06 0.0045857"/>
-      <mass value="1.3904"/>
-      <inertia ixx="0.0050443" ixy="6.668E-07" ixz="3.1856E-05" iyy="0.0045117" iyz="-2.2281E-07" izz="0.0045121"/>
-    </inertial>
-    <visual>
-      <origin rpy="0 0 0" xyz="0 0 0"/>
-      <geometry>
-        <mesh filename="package://rogue/description/meshes/Driving_Right_Link.stl"/>
-      </geometry>
-    </visual>
-    <collision>
-      <origin rpy="0 0 0" xyz="0 0 0"/>
-      <geometry>
-        <mesh filename="package://rogue/description/meshes/Driving_Right_Link.stl"/>
-      </geometry>
-    </collision>
-  </link>
+    <axis xyz="1 0 0"/>
+  </joint>
 </robot>
