Commit message: This sim is launching

File: src/rogue/description/urdf/rogue_des.xacro (robot description, xacro)
@@ -27,5 +27,5 @@
     <origin rpy="0 0 0" xyz="0 0.235 0.11"/>
       <geometry>
-        <mesh filename="package://rogue/description/meshes/base_link.stl"/>
+        <mesh filename="file:///$(find rogue)/description/meshes/base_link.stl"/>
       </geometry>
       <material name="">
@@ -36,8 +36,11 @@
       <origin rpy="0 0 0" xyz="0 0.235 0.11"/>
       <geometry>
-        <mesh filename="package://rogue/description/meshes/base_link.stl"/>
-      </geometry>
-    </collision>
-  </link>
+        <mesh filename="file:///$(find rogue)/description/meshes/base_link.stl"/>
+      </geometry>
+    </collision>
+  </link>
+  <gazebo reference="chassis_link">
+      <material>Gazebo/Gray</material>
+  </gazebo>
   <link name="Steering_Front_Left_Link">
     <inertial>
@@ -49,5 +52,5 @@
       <origin rpy="0 0 0" xyz="0 0 0"/>
       <geometry>
-        <mesh filename="package://rogue/description/meshes/Steering_Front_Left_Link.stl"/>
+        <mesh filename="file:///$(find rogue)/description/meshes/Steering_Front_Left_Link.stl"/>
       </geometry>
       <material name="">
@@ -58,8 +61,11 @@
       <origin rpy="0 0 0" xyz="0 0 0"/>
       <geometry>
-        <mesh filename="package://rogue/description/meshes/Steering_Front_Left_Link.stl"/>
-      </geometry>
-    </collision>
-  </link>
+        <mesh filename="file:///$(find rogue)/description/meshes/Steering_Front_Left_Link.stl"/>
+      </geometry>
+    </collision>
+  </link>
+  <gazebo reference="Steering_Front_Left_Link">
+      <material>Gazebo/Grey</material>
+  </gazebo>
   <joint name="Steering_Front_Left" type="continuous">
     <origin rpy="-1.5789896816345 0 -1.5707963267949" xyz="-0.539929731609329 -0.307999999999972 -0.0838046685206459"/>
@@ -77,5 +83,5 @@
       <origin rpy="0 0 0" xyz="0 0.148 0"/>
       <geometry>
-        <mesh filename="package://rogue/description/meshes/Driving_Front_Left_Link.stl"/>
+        <mesh filename="file:///$(find rogue)/description/meshes/Driving_Front_Left_Link.stl"/>
       </geometry>
       <material name="">
@@ -86,8 +92,11 @@
       <origin rpy="0 0 0" xyz="0 0.148 0"/>
       <geometry>
-        <mesh filename="package://rogue/description/meshes/Driving_Front_Left_Link.stl"/>
-      </geometry>
-    </collision>
-  </link>
+        <mesh filename="file:///$(find rogue)/description/meshes/Driving_Front_Left_Link.stl"/>
+      </geometry>
+    </collision>
+  </link>
+  <gazebo reference="Driving_Front_Left_Link">
+      <material>Gazebo/Red</material>
+  </gazebo>
   <joint name="Driving_Front_Left" type="continuous">
     <origin rpy="0 0 3.14159265358979" xyz="0 ${0.14261211817947+0.148} 0"/>
@@ -105,5 +114,5 @@
       <origin rpy="0 0 0" xyz="0 0 0"/>
       <geometry>
-        <mesh filename="package://rogue/description/meshes/Steering_Front_Right_Link.stl"/>
+        <mesh filename="file:///$(find rogue)/description/meshes/Steering_Front_Right_Link.stl"/>
       </geometry>
       <material name="">
@@ -114,8 +123,11 @@
       <origin rpy="0 0 0" xyz="0 0 0"/>
       <geometry>
-        <mesh filename="package://rogue/description/meshes/Steering_Front_Right_Link.stl"/>
-      </geometry>
-    </collision>
-  </link>
+        <mesh filename="file:///$(find rogue)/description/meshes/Steering_Front_Right_Link.stl"/>
+      </geometry>
+    </collision>
+  </link>
+  <gazebo reference="Steering_Front_Right_Link">
+      <material>Gazebo/Grey</material>
+  </gazebo>
   <joint name="Steering_Front_Right" type="continuous">
     <origin rpy="1.57827537993681 0 1.5707963267949" xyz="-0.539856087012609 0.308000000000008 -0.0842760180023664"/>
@@ -133,5 +145,5 @@
       <origin rpy="0 0 0" xyz="0 -0.148 0"/>
       <geometry>
-        <mesh filename="package://rogue/description/meshes/Driving_Front_Right_Link.stl"/>
+        <mesh filename="file:///$(find rogue)/description/meshes/Driving_Front_Right_Link.stl"/>
       </geometry>
       <material name="">
@@ -142,8 +154,11 @@
       <origin rpy="0 0 0" xyz="0 -0.148 0"/>
       <geometry>
-        <mesh filename="package://rogue/description/meshes/Driving_Front_Right_Link.stl"/>
-      </geometry>
-    </collision>
-  </link>
+        <mesh filename="file:///$(find rogue)/description/meshes/Driving_Front_Right_Link.stl"/>
+      </geometry>
+    </collision>
+  </link>
+  <gazebo reference="Driving_Front_Right_Link">
+      <material>Gazebo/Red</material>
+  </gazebo>
   <joint name="Driving_Front_Right" type="continuous">
     <origin rpy="0 0 3.14159265358979" xyz="0 ${-0.142741590881956-0.148} 0"/>
@@ -161,17 +176,20 @@
       <origin rpy="0 0 0" xyz="0 0 0"/>
       <geometry>
-        <mesh filename="package://rogue/description/meshes/Driving_Left_Link.stl"/>
-      </geometry>
-      <material name="">
-        <color rgba="0.792156862745098 0.819607843137255 0.933333333333333 1"/>
-      </material>
-    </visual>
-    <collision>
-      <origin rpy="0 0 0" xyz="0 0 0"/>
-      <geometry>
-        <mesh filename="package://rogue/description/meshes/Driving_Left_Link.stl"/>
-      </geometry>
-    </collision>
-  </link>
+        <mesh filename="file:///$(find rogue)/description/meshes/Driving_Left_Link.stl"/>
+      </geometry>
+      <material name="">
+        <color rgba="0.792156862745098 0.819607843137255 0.933333333333333 1"/>
+      </material>
+    </visual>
+    <collision>
+      <origin rpy="0 0 0" xyz="0 0 0"/>
+      <geometry>
+        <mesh filename="file:///$(find rogue)/description/meshes/Driving_Left_Link.stl"/>
+      </geometry>
+    </collision>
+  </link>
+  <gazebo reference="Driving_Left_Link">
+      <material>Gazebo/Red</material>
+  </gazebo>
   <joint name="Driving_Left" type="continuous">
     <origin rpy="1.5707963267949 0 1.5707963267949" xyz="0.535731179493507 -0.172500000000432 -0.38861768424532"/>
@@ -189,17 +207,20 @@
       <origin rpy="0 0 0" xyz="0 0 0"/>
       <geometry>
-        <mesh filename="package://rogue/description/meshes/Driving_Right_Link.stl"/>
-      </geometry>
-      <material name="">
-        <color rgba="0.792156862745098 0.819607843137255 0.933333333333333 1"/>
-      </material>
-    </visual>
-    <collision>
-      <origin rpy="0 0 0" xyz="0 0 0"/>
-      <geometry>
-        <mesh filename="package://rogue/description/meshes/Driving_Right_Link.stl"/>
-      </geometry>
-    </collision>
-  </link>
+        <mesh filename="file:///$(find rogue)/description/meshes/Driving_Right_Link.stl"/>
+      </geometry>
+      <material name="">
+        <color rgba="0.792156862745098 0.819607843137255 0.933333333333333 1"/>
+      </material>
+    </visual>
+    <collision>
+      <origin rpy="0 0 0" xyz="0 0 0"/>
+      <geometry>
+        <mesh filename="file:///$(find rogue)/description/meshes/Driving_Right_Link.stl"/>
+      </geometry>
+    </collision>
+  </link>
+  <gazebo reference="Driving_Right_Link">
+      <material>Gazebo/Red</material>
+  </gazebo>
   <joint name="Driving_Right" type="continuous">
     <origin rpy="-1.5707963267949 0 -1.5707963267949" xyz="0.536022919102346 0.17249999999957 -0.388234906342967"/>
